File: DemoShield/DemoShield.kicad_pcb (KiCad board)
At the start: 2 copper layers, 68.6 x 53.3 mm, 22 parts, among them P1 Power, P2 Analog, P3 Digital, P4 Digital, P5 CONN_01X01, P6 CONN_01X01, P7 CONN_01X01, P8 CONN_01X01, U1 gas_sensor, U2 LTC1050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

Commit message: shield V2
Routing:
- net /12(MISO): track 43.9 -> 40.2 mm
Changed lines of the file:
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@@
     (thickness 1.6)
     (drawings 27)
-    (tracks 76)
+    (tracks 78)
     (zones 0)
     (modules 22)
@@
   (segment (start 165.608 99.695) (end 169.418 99.695) (width 0.8) (layer B.Cu) (net 27))
   (segment (start 166.878 97.155) (end 169.418 97.155) (width 0.8) (layer B.Cu) (net 28))
-  (segment (start 144.018 90.805) (end 160.528 90.805) (width 0.8) (layer B.Cu) (net 28))
   (segment (start 160.528 90.805) (end 166.878 97.155) (width 0.8) (layer B.Cu) (net 28))
-  (segment (start 142.494 75.565) (end 142.494 89.281) (width 0.8) (layer B.Cu) (net 28))
-  (segment (start 142.494 89.281) (end 144.018 90.805) (width 0.8) (layer B.Cu) (net 28))
+  (segment (start 142.494 75.565) (end 142.494 82.931) (width 0.8) (layer B.Cu) (net 28))
+  (segment (start 142.494 82.931) (end 144.018 84.455) (width 0.8) (layer B.Cu) (net 28))
+  (segment (start 144.018 84.455) (end 147.828 84.455) (width 0.8) (layer B.Cu) (net 28))
+  (segment (start 147.828 84.455) (end 154.178 90.805) (width 0.8) (layer B.Cu) (net 28))
+  (segment (start 154.178 90.805) (end 160.528 90.805) (width 0.8) (layer B.Cu) (net 28))
   (segment (start 145.034 81.661) (end 145.288 81.915) (width 0.8) (layer B.Cu) (net 29))
   (segment (start 145.034 75.565) (end 145.034 81.661) (width 0.8) (layer B.Cu) (net 29))
@@
   (zone (net 2) (net_name GND) (layer B.Cu) (hatch edge 0.508)
     (connect_pads (clearance 0.508))
+    (min_thickness 0.254)
+    (fill yes (arc_segments 16) (thermal_gap 0.508) (thermal_bridge_width 0.508))
+    (polygon
+      (pts
+        (xy 110.998 73.025) (xy 175.768 73.025) (xy 177.038 74.295) (xy 177.038 85.725) (xy 179.578 88.265)
+        (xy 179.578 121.285) (xy 177.038 123.825) (xy 177.038 126.365) (xy 110.998 126.365)
+      )
+    )
+  )
+  (zone (net 2) (net_name GND) (layer B.Cu) (hatch edge 0.508)
+    (connect_pads (clearance 0.508))
+    (min_thickness 0.254)
+    (fill yes (arc_segments 16) (thermal_gap 0.508) (thermal_bridge_width 0.508))
+    (polygon
+      (pts
+        (xy 110.998 73.025) (xy 175.768 73.025) (xy 177.038 74.295) (xy 177.038 85.725) (xy 179.578 88.265)
+        (xy 179.578 121.285) (xy 177.038 123.825) (xy 177.038 126.365) (xy 110.998 126.365)
+      )
+    )
+  )
+  (zone (net 2) (net_name GND) (layer B.Cu) (hatch edge 0.508)
+    (connect_pads (clearance 0.508))
